Commit message: Add scaling support to URDF and update Gazebo plugins
Introduces a 'scale' argument and scale_factor property to the URDF Xacro files, updating all relevant dimensions and masses to support model scaling. Updates Gazebo plugin code to use ignition::math types and new Gazebo API methods, and fixes Python 3 print compatibility in control scripts. Also adds UUID library detection in CMake and cleans up launch file formatting. File permissions for several scripts and configs were normalized from 755 to 644.

File: morus_description/urdf/morus.urdf.xacro (robot description, xacro)
@@ -2,19 +2,22 @@
 <robot name="morus" xmlns:xacro="http://ros.org/wiki/xacro">
   <!-- Properties -->
+  <xacro:arg name="name" default="drone" />
+  <xacro:arg name="scale" default="1.0" />
+  <xacro:property name="scale_factor" value="$(arg scale)" />
   <xacro:property name="rotor_velocity_slowdown_sim" value="10" />
   <xacro:arg name="custom_mesh_file" default="morus_uav_final.dae" />
   <xacro:property name="mesh_file" value="$(arg custom_mesh_file)" />
   <xacro:property name="mesh_file_mass" value="MORUS_mass.dae" />
-  <xacro:property name="mass" value="30" />  <!-- [kg] -->
-   <xacro:property name="body_width" value="0.35" /> <!-- 0.1 [m] -->
-  <xacro:property name="body_height" value="0.15" /> <!--0.2 [m] -->
-  <xacro:property name="mass_rotor" value="0.2" /> <!-- [kg] -->
-  <xacro:property name="arm_length" value="0.65" /> <!-- [m] -->
-  <xacro:property name="arm_offset" value="0.175" /> <!-- [m] -->
-  <xacro:property name="prop_ver_offset" value="0.15" /> <!-- [m] -->
-  <xacro:property name="prop_long_offset" value="0.07" /> <!-- [m] -->
-  <xacro:property name="radius_rotor" value="0.33" /> <!-- [m] -->
-  <xacro:property name="motor_constant" value="0.000456874" /> <!-- [kg*m/s^2] -->
-  <xacro:property name="moment_constant" value="0.025" /> <!-- [m] -->
+  <xacro:property name="mass" value="${1 * scale_factor}" />  <!-- [kg] -->
+  <xacro:property name="body_width" value="${0.35 * scale_factor}" /> <!-- [m] -->
+  <xacro:property name="body_height" value="${0.15 * scale_factor}" /> <!-- [m] -->
+  <xacro:property name="mass_rotor" value="${0.2 * scale_factor}" /> <!-- [kg] -->
+  <xacro:property name="arm_length" value="${0.65 * scale_factor}" /> <!-- [m] -->
+  <xacro:property name="arm_offset" value="${0.175 * scale_factor}" /> <!-- [m] -->
+  <xacro:property name="prop_ver_offset" value="${0.15 * scale_factor}" /> <!-- [m] -->
+  <xacro:property name="prop_long_offset" value="${0.07 * scale_factor}" /> <!-- [m] -->
+  <xacro:property name="radius_rotor" value="${0.33 * scale_factor}" /> <!-- [m] -->
+  <xacro:property name="motor_constant" value="${0.000456874 * scale_factor}" /> <!-- [kg*m/s^2] -->
+  <xacro:property name="moment_constant" value="${0.025 * scale_factor}" /> <!-- [m] -->
   <xacro:property name="time_constant_up" value="0.2" /> <!-- [s] -->
   <xacro:property name="time_constant_down" value="0.2" /> <!-- [s] -->
@@ -22,9 +25,9 @@
   <xacro:property name="rotor_drag_coefficient" value="0.0" /> <!--8.06428e-03-->
   <xacro:property name="rolling_moment_coefficient" value="0.00001" />
-  <xacro:property name="movable_mass_mass" value="1" />
-  <xacro:property name="movable_mass_dimension" value="0.08" />
-  <xacro:property name="movable_mass_offset" value="0.05" />
-  <xacro:property name="imu_mass" value="0.02"/>
-  <xacro:property name="imu_size" value="0.01"/>
+  <xacro:property name="movable_mass_mass" value="${1 * scale_factor}" />
+  <xacro:property name="movable_mass_dimension" value="${0.08 * scale_factor}" />
+  <xacro:property name="movable_mass_offset" value="${0.05 * scale_factor}" />
+  <xacro:property name="imu_mass" value="${0.02 * scale_factor}"/>
+  <xacro:property name="imu_size" value="${0.01 * scale_factor}"/>
   <xacro:property name="sin45" value="0.7071" />
   <xacro:property name="cos45" value="0.7071" />
@@ -68,5 +71,6 @@
     body_height="${body_height}"
     mesh_file="${mesh_file}"
-    mesh_file_mass="${mesh_file_mass}">
+    mesh_file_mass="${mesh_file_mass}"
+    scale_factor="${scale_factor}">
     <xacro:insert_block name="body_inertia" />
   </xacro:multirotor_base_macro>
@@ -230,9 +234,9 @@
       parent="base_link"
       gear_num = "1"
-      mass = "1e-6"
-      dim_x = "0.12"
-      dim_y = "0.04"
-      dim_z = "0.0001">
-      <origin xyz="0 -0.7 -0.275" rpy="0 0 0" />
+      mass = "${1e-6 * scale_factor}"
+      dim_x = "${0.12 * scale_factor}"
+      dim_y = "${0.04 * scale_factor}"
+      dim_z = "${0.0001 * scale_factor}">
+      <origin xyz="0 ${-0.7 * scale_factor} ${-0.275 * scale_factor}" rpy="0 0 0" />
       <xacro:insert_block name="land_gear_inertia"/>
   </xacro:landing_gear>
@@ -240,9 +244,9 @@
       parent="base_link"
       gear_num = "2"
-      mass = "1e-6"
-      dim_x = "0.12"
-      dim_y = "0.04"
-      dim_z = "0.0001">
-      <origin xyz="0 0.7 -0.275" rpy="0 0 0" />
+      mass = "${1e-6 * scale_factor}"
+      dim_x = "${0.12 * scale_factor}"
+      dim_y = "${0.04 * scale_factor}"
+      dim_z = "${0.0001 * scale_factor}">
+      <origin xyz="0 ${0.7 * scale_factor} ${-0.275 * scale_factor}" rpy="0 0 0" />
       <xacro:insert_block name="land_gear_inertia"/>
   </xacro:landing_gear>
@@ -250,9 +254,9 @@
       parent="base_link"
       gear_num = "3"
-      mass = "1e-6"
-      dim_x = "0.12"
-      dim_y = "0.04"
-      dim_z = "0.0001">
-      <origin xyz="-0.7 0 -0.275" rpy="0 0 1.57" />
+      mass = "${1e-6 * scale_factor}"
+      dim_x = "${0.12 * scale_factor}"
+      dim_y = "${0.04 * scale_factor}"
+      dim_z = "${0.0001 * scale_factor}">
+      <origin xyz="${-0.7 * scale_factor} 0 ${-0.275 * scale_factor}" rpy="0 0 1.57" />
       <xacro:insert_block name="land_gear_inertia"/>
   </xacro:landing_gear>
@@ -260,10 +264,16 @@
       parent="base_link"
       gear_num = "4"
-      mass = "1e-6"
-      dim_x = "0.12"
-      dim_y = "0.04"
-      dim_z = "0.0001">
-      <origin xyz="0.7 0.0 -0.275" rpy="0 0 1.57" />
-      <xacro:insert_block name="land_gear_inertia"/>
-  </xacro:landing_gear>
+      mass = "${1e-6 * scale_factor}"
+      dim_x = "${0.12 * scale_factor}"
+      dim_y = "${0.04 * scale_factor}"
+      dim_z = "${0.0001 * scale_factor}">
+      <origin xyz="${0.7 * scale_factor} 0.0 ${-0.275 * scale_factor}" rpy="0 0 1.57" />
+      <xacro:insert_block name="land_gear_inertia"/>
+  </xacro:landing_gear>
+  <!-- Se nel file c'è una chiamata alla macro camera_macro, aggiorna per passare scale_factor -->
+  <!-- Esempio (aggiungi questo codice se non esiste la chiamata alla macro camera): -->
+  <!-- <xacro:camera_macro
+    robot_namespace="$(arg name)"
+    scale_factor="${scale_factor}">
+  </xacro:camera_macro> -->
 </robot>

File: morus_description/urdf/multirotor_base.urdf.xacro (robot description, xacro)
@@ -3,5 +3,5 @@
   <!-- Main multirotor link -->
   <xacro:macro name="multirotor_base_macro"
-    params="robot_namespace mass body_width body_height mesh_file mesh_file_mass *inertia">
+    params="robot_namespace mass body_width body_height mesh_file mesh_file_mass scale_factor *inertia">
     <link name="base_link"></link>
     <joint name="base_joint" type="fixed">
@@ -17,8 +17,8 @@
       </inertial>
       <visual>
-        <origin xyz="0 0 -0.65" rpy="0 0 0" />
+        <origin xyz="0 0 ${-0.65 * scale_factor}" rpy="0 0 0" />
         <geometry>
           <mesh filename="package://morus_description/meshes/${mesh_file}"
-            scale="0.001 0.001 0.001" />
+            scale="${0.001 * scale_factor} ${0.001 * scale_factor} ${0.001 * scale_factor}" />
           <!--box size="${body_width} ${body_width} ${body_height}"/--> <!-- [m] [m] [m] -->
         </geometry>
@@ -36,5 +36,5 @@
         <inertia ixx="0.00001" ixy="0.0" ixz="0.0" iyy="0.00001" iyz="0.0"
           izz="0.00001" />
-        <mass value="0.01" />  <!-- [kg] -->
+        <mass value="${0.01 * scale_factor}" />  <!-- [kg] -->
         <origin xyz="0 0 0" rpy="0 0 0" />
       </inertial>
@@ -64,5 +64,5 @@
       <parent link="${parent}"/>
       <child link="movable_mass_${mass_number}"/>
-      <limit lower="-0.3" upper="0.3" effort="10000" velocity="20"/>
+      <limit lower="${-0.3 * scale_factor}" upper="${0.3 * scale_factor}" effort="10000" velocity="20"/>
       <dynamics damping="10" />  <!--friction="0.1" used only in Gazebo >= 5.0, damping is the viscous friction damping,
        i.e. Ft = damping * v -->
@@ -71,5 +71,5 @@
       <visual>
         <!--origin rpy="0 0 ${orientation}" xyz="0 0 ${0*movable_mass_dimension/2}"/-->
-        <origin rpy="0 0 ${orientation}" xyz="0 0 -0.05"/>
+        <origin rpy="0 0 ${orientation}" xyz="0 0 ${-0.05 * scale_factor}"/>
         <geometry>
           <!--mesh filename="package://morus_description/meshes/${mesh_file_mass}"
@@ -117,5 +117,5 @@
           <!-- <cylinder length="0.005" radius="${radius_rotor}"/> --> <!-- [m] -->
           <mesh filename="package://morus_description/meshes/propeller_${direction}.dae"
-            scale="0.0025 0.0025 0.0025" />
+            scale="${0.0025 * scale_factor} ${0.0025 * scale_factor} ${0.0025 * scale_factor}" />
           <!-- <box size="${2*radius_rotor} 0.01 0.005"/> -->
         </geometry>
@@ -123,5 +123,5 @@
       <collision>
         <geometry>
-          <cylinder length="0.005" radius="${radius_rotor}" /> <!-- [m] -->
+          <cylinder length="${0.005 * scale_factor}" radius="${radius_rotor}" /> <!-- [m] -->
         </geometry>
       </collision>
@@ -190,9 +190,9 @@
   </xacro:macro>
    <!-- camera -->
-  <xacro:macro name="camera_macro" params="robot_namespace">
+  <xacro:macro name="camera_macro" params="robot_namespace scale_factor">
     <!-- joint -->
     <joint name="camera_joint" type="fixed">
       <axis xyz="0 1 0" />
-      <origin xyz="0 0 0.2" rpy="0 0 0" />
+      <origin xyz="0 0 ${0.2 * scale_factor}" rpy="0 0 0" />
       <parent link="base_link" />
       <child link="camera_link" />
@@ -203,16 +203,16 @@
         <origin xyz="0 0 0" rpy="0 0 0" />
         <geometry>
-          <box size="0.1 0.1 0.1" />
-        </geometry>
-      </collision>
-      <visual>
-        <origin xyz="0 0 0" rpy="0 0 0" />
-        <geometry>
-          <box size="0.1 0.1 0.1" />
+          <box size="${0.1 * scale_factor} ${0.1 * scale_factor} ${0.1 * scale_factor}" />
+        </geometry>
+      </collision>
+      <visual>
+        <origin xyz="0 0 0" rpy="0 0 0" />
+        <geometry>
+          <box size="${0.1 * scale_factor} ${0.1 * scale_factor} ${0.1 * scale_factor}" />
         </geometry>
         <material name="red" />
       </visual>
       <inertial>
-        <mass value="1e-5" />
+        <mass value="${1e-5 * scale_factor}" />
         <origin xyz="0 0 0" rpy="0 0 0" />
         <inertia ixx="1e-6" ixy="0" ixz="0" iyy="1e-6" iyz="0" izz="1e-6" />
