Commit message: Add tf_prefix and base_link_name support to xacro files
Introduces tf_prefix and base_link_name arguments and properties to all major URDF xacro files for improved namespace flexibility. Updates macros and link/joint definitions to use these properties, ensuring correct namespacing for multi-robot simulation and integration. Adds new drone_sim.xacro for simulation-specific configuration.

File: morus_description/urdf/morus.base.urdf.xacro (robot description, xacro)
@@ -1,4 +1,8 @@
 <?xml version="1.0"?>
 <robot name="morus" xmlns:xacro="http://ros.org/wiki/xacro">
+  <xacro:arg name="base_link_name" default="base_link" />
+  <xacro:arg name="tf_prefix" default="" />
+  <xacro:property name="tf_prefix" value="$(arg tf_prefix)" />
+  <xacro:property name="base_link_name" value="$(arg base_link_name)" />
   <!-- Properties -->
   <xacro:property name="rotor_velocity_slowdown_sim" value="10" />
@@ -65,5 +69,8 @@
     body_height="${body_height}"
     mesh_file="${mesh_file}"
-    mesh_file_mass="${mesh_file_mass}">
+    mesh_file_mass="${mesh_file_mass}"
+    scale_factor="1.0"
+    base_link_name="${base_link_name}"
+    tf_prefix="${tf_prefix}">
     <xacro:insert_block name="body_inertia" />
   </xacro:multirotor_base_macro>
@@ -76,5 +83,6 @@
   </xacro:property>
   <xacro:landing_gear
-      parent="base_link"
+      parent="${base_link_name}"
+      tf_prefix="${tf_prefix}"
       gear_num = "1"
       mass = "1e-6"
@@ -86,5 +94,6 @@
   </xacro:landing_gear>
   <xacro:landing_gear
-      parent="base_link"
+      parent="${base_link_name}"
+      tf_prefix="${tf_prefix}"
       gear_num = "2"
       mass = "1e-6"

File: morus_description/urdf/multirotor_base.urdf.xacro (robot description, xacro)
@@ -1,14 +1,27 @@
 <?xml version="1.0"?>
 <robot xmlns:xacro="http://ros.org/wiki/xacro">
+  <!-- Helper property to create link names with tf_prefix -->
+  <xacro:property name="link_prefix" value="${tf_prefix}" />
   <!-- Main multirotor link -->
   <xacro:macro name="multirotor_base_macro"
-    params="robot_namespace mass body_width body_height mesh_file mesh_file_mass scale_factor *inertia">
-    <link name="base_link"></link>
+    params="robot_namespace mass body_width body_height mesh_file mesh_file_mass scale_factor base_link_name tf_prefix *inertia">
+    <!-- Create link names with tf_prefix -->
+    <xacro:if value="${tf_prefix != ''}">
+      <xacro:property name="prefixed_base_link" value="${tf_prefix}/${base_link_name}" />
+      <xacro:property name="prefixed_base_link_inertia" value="${tf_prefix}/${base_link_name}_inertia" />
+      <xacro:property name="prefixed_imu_link" value="${tf_prefix}/imu_link" />
+    </xacro:if>
+    <xacro:unless value="${tf_prefix != ''}">
+      <xacro:property name="prefixed_base_link" value="${base_link_name}" />
+      <xacro:property name="prefixed_base_link_inertia" value="${base_link_name}_inertia" />
+      <xacro:property name="prefixed_imu_link" value="imu_link" />
+    </xacro:unless>
+    <link name="${prefixed_base_link}"></link>
     <joint name="base_joint" type="fixed">
       <origin xyz="0 0 0" rpy="0 0 0" />
-      <parent link="base_link" />
-      <child link="base_link_inertia" />
-    </joint>
-    <link name="base_link_inertia">
+      <parent link="${prefixed_base_link}" />
+      <child link="${prefixed_base_link_inertia}" />
+    </joint>
+    <link name="${prefixed_base_link_inertia}">
       <inertial>
         <mass value="${mass}" />  <!-- [kg] -->
@@ -32,5 +45,5 @@
     </link>
     <!-- IMU -->
-    <link name="imu_link">
+    <link name="${prefixed_imu_link}">
       <inertial>
         <inertia ixx="0.00001" ixy="0.0" ixz="0.0" iyy="0.00001" iyz="0.0"
@@ -43,6 +56,6 @@
     <joint name="imu_joint" type="revolute">
       <!--origin xyz="0 0 0" rpy="3.1416 0 0" / -->
-      <parent link="base_link" />
-      <child link="imu_link" />
+      <parent link="${prefixed_base_link}" />
+      <child link="${prefixed_imu_link}" />
       <limit upper="0" lower="0" effort="0" velocity="0" />
     </joint>
@@ -51,5 +64,5 @@
       <plugin filename="librotors_gazebo_multirotor_base_plugin.so" name="rosbag">
         <robotNamespace>$(arg name)</robotNamespace>
-        <linkName>base_link</linkName>
+        <linkName>${prefixed_base_link}</linkName>
         <rotorVelocitySlowdownSim>${rotor_velocity_slowdown_sim}</rotorVelocitySlowdownSim>
       </plugin>
@@ -58,15 +71,24 @@
   <!-- Macro file for movable mass. It defines joint between mass and stick, and link which defines actual mass. Stick
   is defined in other macro file-->
-  <xacro:macro name="movable_mass" params="mass_number parent mass dimension color x_axis y_axis z_axis orientation *origin *inertia">
+  <xacro:macro name="movable_mass" params="mass_number parent tf_prefix mass dimension color x_axis y_axis z_axis orientation *origin *inertia">
+    <!-- Create prefixed link name -->
+    <xacro:if value="${tf_prefix != ''}">
+      <xacro:property name="prefixed_movable_mass" value="${tf_prefix}/movable_mass_${mass_number}" />
+      <xacro:property name="prefixed_parent" value="${tf_prefix}/${parent}" />
+    </xacro:if>
+    <xacro:unless value="${tf_prefix != ''}">
+      <xacro:property name="prefixed_movable_mass" value="movable_mass_${mass_number}" />
+      <xacro:property name="prefixed_parent" value="${parent}" />
+    </xacro:unless>
     <joint name="stick_to_movable_mass_${mass_number}" type="prismatic">
       <xacro:insert_block name="origin"/>
       <axis xyz="${x_axis} ${y_axis} ${z_axis}"/>
-      <parent link="${parent}"/>
-      <child link="movable_mass_${mass_number}"/>
+      <parent link="${prefixed_parent}"/>
+      <child link="${prefixed_movable_mass}"/>
       <limit lower="${-0.3 * scale_factor}" upper="${0.3 * scale_factor}" effort="10000" velocity="20"/>
       <dynamics damping="10" />  <!--friction="0.1" used only in Gazebo >= 5.0, damping is the viscous friction damping,
        i.e. Ft = damping * v -->
     </joint>
-    <link name="movable_mass_${mass_number}">
+    <link name="${prefixed_movable_mass}">
       <visual>
         <!--origin rpy="0 0 ${orientation}" xyz="0 0 ${0*movable_mass_dimension/2}"/-->
@@ -90,5 +112,5 @@
       </inertial>
     </link>
-    <gazebo reference="movable_mass_${mass_number}">
+    <gazebo reference="${prefixed_movable_mass}">
       <material>Gazebo/${color}</material>
     </gazebo>
@@ -96,5 +118,14 @@
   <!-- Rotor joint and link -->
   <xacro:macro name="vertical_rotor"
-    params="robot_namespace suffix direction motor_constant moment_constant parent mass_rotor radius_rotor time_constant_up time_constant_down max_rot_velocity motor_number rotor_drag_coefficient rolling_moment_coefficient color *origin *inertia">
+    params="robot_namespace suffix direction motor_constant moment_constant parent tf_prefix mass_rotor radius_rotor time_constant_up time_constant_down max_rot_velocity motor_number rotor_drag_coefficient rolling_moment_coefficient color *origin *inertia">
+    <!-- Create prefixed link names -->
+    <xacro:if value="${tf_prefix != ''}">
+      <xacro:property name="prefixed_rotor" value="${tf_prefix}/rotor_${motor_number}" />
+      <xacro:property name="prefixed_parent" value="${tf_prefix}/${parent}" />
+    </xacro:if>
+    <xacro:unless value="${tf_prefix != ''}">
+      <xacro:property name="prefixed_rotor" value="rotor_${motor_number}" />
+      <xacro:property name="prefixed_parent" value="${parent}" />
+    </xacro:unless>
     <joint name="rotor_${motor_number}_joint" type="continuous">
       <xacro:insert_block name="origin" />
@@ -102,11 +133,11 @@
       <!-- TODO(ff): not currently set because it's not yet supported -->
       <!-- <limit effort="2000" velocity="${max_rot_velocity}" /> -->
-      <parent link="${parent}" />
-      <child link="rotor_${motor_number}" />
+      <parent link="${prefixed_parent}" />
+      <child link="${prefixed_rotor}" />
     </joint>
     <!-- TODO(ff): not currently set because it's not yet supported -->
     <!-- <gazebo reference="rotor_${motor_number}_joint"> <axis> <xyz>0 0 1</xyz>
       <limit> <velocity> ${max_rot_velocity} </velocity> </limit> </axis> </gazebo> -->
-    <link name="rotor_${motor_number}">
+    <link name="${prefixed_rotor}">
       <inertial>
         <mass value="${mass_rotor}" /> <!-- [kg] -->
@@ -130,5 +161,5 @@
       <plugin name="${suffix}_motor_model" filename="librotors_gazebo_motor_model.so">
         <jointName>rotor_${motor_number}_joint</jointName>
-        <linkName>rotor_${motor_number}</linkName>
+        <linkName>${prefixed_rotor}</linkName>
         <turningDirection>${direction}</turningDirection>
         <timeConstantUp>${time_constant_up}</timeConstantUp>
@@ -145,5 +176,5 @@
       </plugin>
     </gazebo>
-    <gazebo reference="rotor_${motor_number}">
+    <gazebo reference="${prefixed_rotor}">
       <material>Gazebo/${color}</material>
     </gazebo>
@@ -162,12 +193,21 @@
     </transmission>
   </xacro:macro>
-  <xacro:macro name="landing_gear" params="gear_num parent mass dim_x dim_y dim_z *origin *inertia">
+  <xacro:macro name="landing_gear" params="gear_num parent tf_prefix mass dim_x dim_y dim_z *origin *inertia">
+    <!-- Create prefixed link names -->
+    <xacro:if value="${tf_prefix != ''}">
+      <xacro:property name="prefixed_landing_gear" value="${tf_prefix}/land_gear_${gear_num}" />
+      <xacro:property name="prefixed_parent" value="${tf_prefix}/${parent}" />
+    </xacro:if>
+    <xacro:unless value="${tf_prefix != ''}">
+      <xacro:property name="prefixed_landing_gear" value="land_gear_${gear_num}" />
+      <xacro:property name="prefixed_parent" value="${parent}" />
+    </xacro:unless>
     <joint name="land_gear_${gear_num}" type="fixed">
       <xacro:insert_block name="origin"/>
       <axis xyz="0 0 1"/>
-      <parent link="${parent}"/>
-      <child link="land_gear_${gear_num}"/>
-    </joint>
-    <link name="land_gear_${gear_num}">
+      <parent link="${prefixed_parent}"/>
+      <child link="${prefixed_landing_gear}"/>
+    </joint>
+    <link name="${prefixed_landing_gear}">
       <!--visual>
         <origin rpy="0 0 0" xyz="0 0 0"/>
@@ -190,14 +230,23 @@
   </xacro:macro>
    <!-- camera -->
-  <xacro:macro name="camera_macro" params="robot_namespace scale_factor">
+  <xacro:macro name="camera_macro" params="robot_namespace scale_factor base_link_name tf_prefix">
+    <!-- Create prefixed link names -->
+    <xacro:if value="${tf_prefix != ''}">
+      <xacro:property name="prefixed_camera_link" value="${tf_prefix}/camera_link" />
+      <xacro:property name="prefixed_base_link" value="${tf_prefix}/${base_link_name}" />
+    </xacro:if>
+    <xacro:unless value="${tf_prefix != ''}">
+      <xacro:property name="prefixed_camera_link" value="camera_link" />
+      <xacro:property name="prefixed_base_link" value="${base_link_name}" />
+    </xacro:unless>
     <!-- joint -->
     <joint name="camera_joint" type="fixed">
       <axis xyz="0 1 0" />
       <origin xyz="0 0 ${0.2 * scale_factor}" rpy="0 0 0" />
-      <parent link="base_link" />
-      <child link="camera_link" />
+      <parent link="${prefixed_base_link}" />
+      <child link="${prefixed_camera_link}" />
     </joint>
     <!-- link -->
-    <link name="camera_link">
+    <link name="${prefixed_camera_link}">
       <collision>
         <origin xyz="0 0 0" rpy="0 0 0" />
@@ -219,5 +268,5 @@
       </inertial>
     </link>
-    <gazebo reference="camera_link">
+    <gazebo reference="${prefixed_camera_link}">
       <sensor type="camera" name="camera1">
         <update_rate>30.0</update_rate>
@@ -245,5 +294,5 @@
           <imageTopicName>image_raw</imageTopicName>
           <cameraInfoTopicName>camera_info</cameraInfoTopicName>
-          <frameName>camera_link</frameName>
+          <frameName>${prefixed_camera_link}</frameName>
           <hackBaseline>0.07</hackBaseline>
           <distortionK1>0.0</distortionK1>
